File: Main/Main.kicad_sch (KiCad schematic)
At the start: 44 parts, among them SW1 RotaryEncoder_Switch_MP, SW2 Switch, U1 Arduino_Pro_Micro, U2 TRRS

Commit message: figured out footprints and stuff
Parts:
- S1, S10, S11, S12, S13, S14, S15, S16, S17, S18, S19, S2, S20, S3, S4, S5, S6, S7, S8, S9: footprint keyswitches:Kailh_socket_PG1350 -> ScottoKeebs_Hotswap:Hotswap_Choc_V1
- SW2: footprint Button_Switch_THT:SW_CW_GPTS203211B -> ScottoKeebs_Components:Button_MJTP1243
- U2: footprint Connector_Audio:Plug_3.5mm_CUI_SP-3541 -> ScottoKeebs_Components:TRRS_PJ-320A
Changed lines of the file:
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@@
 			)
 		)
-		(property "Footprint" "keyswitches:Kailh_socket_PG1350"
+		(property "Footprint" "ScottoKeebs_Hotswap:Hotswap_Choc_V1"
 			(at 77.47 60.96 0)
 			(effects
@@
 			)
 		)
-		(property "Footprint" "keyswitches:Kailh_socket_PG1350"
+		(property "Footprint" "ScottoKeebs_Hotswap:Hotswap_Choc_V1"
 			(at 90.17 72.39 0)
 			(effects
@@
 			)
 		)
-		(property "Footprint" "keyswitches:Kailh_socket_PG1350"
+		(property "Footprint" "ScottoKeebs_Hotswap:Hotswap_Choc_V1"
 			(at 58.42 49.53 0)
 			(effects
@@
 			)
 		)
-		(property "Footprint" "keyswitches:Kailh_socket_PG1350"
+		(property "Footprint" "ScottoKeebs_Hotswap:Hotswap_Choc_V1"
 			(at 90.17 60.96 0)
 			(effects
@@
 			)
 		)
-		(property "Footprint" "keyswitches:Kailh_socket_PG1350"
+		(property "Footprint" "ScottoKeebs_Hotswap:Hotswap_Choc_V1"
 			(at 64.77 60.96 0)
 			(effects
@@
 			)
 		)
-		(property "Footprint" "Button_Switch_THT:SW_CW_GPTS203211B"
+		(property "Footprint" "ScottoKeebs_Components:Button_MJTP1243"
 			(at 128.27 68.58 0)
 			(effects
@@
 			)
 		)
-		(property "Footprint" "keyswitches:Kailh_socket_PG1350"
+		(property "Footprint" "ScottoKeebs_Hotswap:Hotswap_Choc_V1"
 			(at 64.77 72.39 0)
 			(effects
@@
 			)
 		)
-		(property "Footprint" "keyswitches:Kailh_socket_PG1350"
+		(property "Footprint" "ScottoKeebs_Hotswap:Hotswap_Choc_V1"
 			(at 77.47 72.39 0)
 			(effects
@@
 			)
 		)
-		(property "Footprint" "keyswitches:Kailh_socket_PG1350"
+		(property "Footprint" "ScottoKeebs_Hotswap:Hotswap_Choc_V1"
 			(at 83.82 72.39 0)
 			(effects
@@
 			)
 		)
-		(property "Footprint" "Connector_Audio:Plug_3.5mm_CUI_SP-3541"
+		(property "Footprint" "ScottoKeebs_Components:TRRS_PJ-320A"
 			(at 177.8 138.43 0)
 			(effects
@@
 			)
 		)
-		(property "Footprint" "keyswitches:Kailh_socket_PG1350"
+		(property "Footprint" "ScottoKeebs_Hotswap:Hotswap_Choc_V1"
 			(at 71.12 49.53 0)
 			(effects
@@
 			)
 		)
-		(property "Footprint" "keyswitches:Kailh_socket_PG1350"
+		(property "Footprint" "ScottoKeebs_Hotswap:Hotswap_Choc_V1"
 			(at 71.12 60.96 0)
 			(effects
@@
 			)
 		)
-		(property "Footprint" "keyswitches:Kailh_socket_PG1350"
+		(property "Footprint" "ScottoKeebs_Hotswap:Hotswap_Choc_V1"
 			(at 90.17 83.82 0)
 			(effects
@@
 			)
 		)
-		(property "Footprint" "keyswitches:Kailh_socket_PG1350"
+		(property "Footprint" "ScottoKeebs_Hotswap:Hotswap_Choc_V1"
 			(at 77.47 49.53 0)
 			(effects
@@
 			)
 		)
-		(property "Footprint" "keyswitches:Kailh_socket_PG1350"
+		(property "Footprint" "ScottoKeebs_Hotswap:Hotswap_Choc_V1"
 			(at 83.82 83.82 0)
 			(effects
@@
 			)
 		)
-		(property "Footprint" "keyswitches:Kailh_socket_PG1350"
+		(property "Footprint" "ScottoKeebs_Hotswap:Hotswap_Choc_V1"
 			(at 64.77 49.53 0)
 			(effects
@@
 			)
 		)
-		(property "Footprint" "keyswitches:Kailh_socket_PG1350"
+		(property "Footprint" "ScottoKeebs_Hotswap:Hotswap_Choc_V1"
 			(at 90.17 49.53 0)
 			(effects
@@
 			)
 		)
-		(property "Footprint" "keyswitches:Kailh_socket_PG1350"
+		(property "Footprint" "ScottoKeebs_Hotswap:Hotswap_Choc_V1"
 			(at 83.82 49.53 0)
 			(effects
@@
 			)
 		)
-		(property "Footprint" "keyswitches:Kailh_socket_PG1350"
+		(property "Footprint" "ScottoKeebs_Hotswap:Hotswap_Choc_V1"
 			(at 58.42 72.39 0)
 			(effects
@@
 			)
 		)
-		(property "Footprint" "keyswitches:Kailh_socket_PG1350"
+		(property "Footprint" "ScottoKeebs_Hotswap:Hotswap_Choc_V1"
 			(at 71.12 72.39 0)
 			(effects
@@
 			)
 		)
-		(property "Footprint" "keyswitches:Kailh_socket_PG1350"
+		(property "Footprint" "ScottoKeebs_Hotswap:Hotswap_Choc_V1"
 			(at 58.42 60.96 0)
 			(effects
@@
 			)
 		)
-		(property "Footprint" "keyswitches:Kailh_socket_PG1350"
+		(property "Footprint" "ScottoKeebs_Hotswap:Hotswap_Choc_V1"
 			(at 83.82 60.96 0)
 			(effects
