File: Main/Main.kicad_pcb (KiCad board)
At the start: 2 copper layers, 44 parts, among them SW1 RotaryEncoder_Switch_MP, SW2 Switch, U1 Arduino_Pro_Micro, U2 TRRS

Commit message: figured out footprints and stuff
Parts:
- S1, S10, S11, S12, S13, S14, S15, S16, S17, S18, S19, S2, S20, S3, S4, S5, S6, S7, S8, S9: footprint keyswitches:Kailh_socket_PG1350 -> ScottoKeebs_Hotswap:Hotswap_Choc_V1
- SW2: footprint Button_Switch_THT:SW_CW_GPTS203211B -> ScottoKeebs_Components:Button_MJTP1243
- U2: footprint Connector_Audio:Plug_3.5mm_CUI_SP-3541 -> ScottoKeebs_Components:TRRS_PJ-320A
- moved U2 224.1 mm to (283.8, 126.0)
- moved SW2 140.5 mm to (227.0, 60.0)
- moved D20 9.04 mm to (261.5, 139.0)
- moved D1 9.04 mm to (153.5, 80.5)
- moved D10 9.04 mm to (207.5, 82.5)
- moved D11 9.04 mm to (229.0, 99.0)
- moved D12 9.04 mm to (246.0, 100.5)
- moved D13 9.04 mm to (154.0, 113.5)
- moved D14 9.04 mm to (172.0, 113.5)
- moved D15 9.04 mm to (189.5, 105.5)
- moved D16 9.04 mm to (207.5, 99.5)
- moved D17 9.04 mm to (227.5, 115.5)
- moved D18 9.04 mm to (245.0, 117.0)
- moved D19 9.04 mm to (244.0, 136.0)
- moved D2 9.04 mm to (171.5, 80.0)
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Routing:
- net 0 Column: track 0.00 -> 33.6 mm

Commit message: finished left PCB
Parts:
- moved U2 53.2 mm to (280.6, 72.9), turned to -4 degrees
- moved U1 0.47 mm to (273.3, 104.3)
Routing:
- net 1 Column: track 0.00 -> 189.7 mm
- net 2 Column: track 0.00 -> 167.4 mm, vias 0 -> 3
- net 1 Row: track 0.00 -> 155.3 mm, vias 0 -> 4
- net 0 Column: track 33.6 -> 186.8 mm, vias 0 -> 1
- net 2 Row: track 0.00 -> 151.4 mm, vias 0 -> 4
- net 0 Row: track 0.00 -> 139.1 mm
- net GND: track 0.00 -> 135.6 mm, vias 0 -> 1
- net 3 Column: track 0.00 -> 127.2 mm, vias 0 -> 5
- net 5 Column: track 0.00 -> 120.9 mm, vias 0 -> 3
- net 4 Column: track 0.00 -> 118.0 mm, vias 0 -> 5
- net 3 Row: track 0.00 -> 72.4 mm, vias 0 -> 1
- net RST: track 0.00 -> 55.6 mm, vias 0 -> 2
- net SCL: track 0.00 -> 44.2 mm, vias 0 -> 3
- net Net-(U1-A3/PF4): track 0.00 -> 35.3 mm, vias 0 -> 2
- net SDA: track 0.00 -> 27.0 mm, vias 0 -> 3
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Other:
- board outline added: 140.2 x 97.8 mm
